File: Design/IndoorSensor/IndoorSensor.kicad_pcb (KiCad board)
At the start: 2 copper layers, 49.5 x 48.3 mm, 17 parts, among them J1 Conn_01x04_Pin, J2 Conn_01x06_Pin, J3 Conn_01x04_Pin, U1 MH-Z19B, U3 WeMos_D1_mini, U4 module_bme280_alt

Commit message: Fix minor issues before production
Routing:
- net SCL: track 70.0 -> 65.3 mm
- net SDA: track 58.2 -> 61.5 mm
- net GPIO13: track 16.9 -> 17.7 mm
- net GPIO12: track 20.5 -> 21.2 mm
- net +3V3: track 9.72 -> 10.5 mm
- net GPIO15: track 13.3 -> 14.1 mm
